File: KicadJE_PocketOperator_TDA1308Amp/KicadJE_PocketOperator_TDA1308Amp.kicad_pcb (KiCad board)
At the start: 2 copper layers, 71.1 x 45.7 mm, 31 parts, among them J101 In 1 + Sync, J102 In 2, J103 In 3, J104 Out Stereo, J105 Sync1, J106 Sync2, SW102 SW_Push_DPDT

Commit message: Logo etc
TDA symbol PSU GND swapped
New logos
Parts:
- added G***: LOGO, AJ_2025_Library:Johansen_engineering_logo_25mm_front_neg5, F.Cu at (87.4, 73.7)
- added G***: LOGO, AJ_2025_Library:OPERATOR_25mm, F.Cu at (113.0, 43.5)
- added G***: LOGO, AJ_2025_Library:TE_Side_45mm, B.Cu at (114.1, 62.6)
- added REF**: Mounting_Wuerth_WA-SMST-4.5mm_H2mm_9774020982, Mounting_Wuerth:Mounting_Wuerth_WA-SMST-4.5mm_H2mm_9774020982, F.Cu at (141.7, 70.6)
- moved JP105 17.3 mm to (99.3, 35.0)
- moved JP106 17.3 mm to (99.3, 37.5)
- moved C101 6.99 mm to (123.9, 64.0), turned to 0 degrees
- moved JP101 3.51 mm to (127.3, 48.3)
- moved JP102 3.51 mm to (127.3, 45.8)
- moved JP103 3.51 mm to (127.3, 37.6)
- moved JP104 3.51 mm to (127.3, 35.0)
- moved SW102 0.61 mm to (101.6, 51.9)
- moved JP107 0.59 mm to (100.6, 54.7)
- moved U101 0.50 mm to (119.4, 60.3)
- moved D101 0.32 mm to (106.1, 49.2)
- moved R101 0.32 mm to (102.3, 49.2)
Other:
- board text added: "ON"

Commit message: Update KicadJE_PocketOperator_TDA1308Amp.kicad_pcb
update TDA 1308 PWR correction
Connections:
- U101 pad 7: +3V8 -> GND
- U101 pad 8: GND -> +3V8
Changed lines of the file:
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@@
 			(remove_unused_layers no)
 			(roundrect_rratio 0.15)
-			(net 22 "+3V8")
-			(pinfunction "Vcc")
+			(net 2 "GND")
+			(pinfunction "GND")
 			(pintype "power_in")
 		)
@@
 			(remove_unused_layers no)
 			(roundrect_rratio 0.15)
-			(net 2 "GND")
-			(pinfunction "GND")
+			(net 22 "+3V8")
+			(pinfunction "Vcc")
 			(pintype "power_in")
 		)

Commit message: Routed
Parts:
- turned JP101 to 180 degrees
- turned JP102 to 180 degrees
Routing:
- net InL: track 0.00 -> 56.3 mm
- net In1L: track 0.00 -> 46.0 mm
- net Net-(JP102-B): track 0.00 -> 44.9 mm
- net InR: track 0.00 -> 39.4 mm
- net Net-(JP101-B): track 0.00 -> 38.2 mm
- net +3V8: track 0.00 -> 35.7 mm
- net In1R: track 0.00 -> 26.1 mm
- net +BATT: track 0.00 -> 25.6 mm
- net Out3L: track 0.00 -> 17.8 mm
- net Out2L: track 0.00 -> 17.5 mm
- net Out1L: track 0.00 -> 17.5 mm
- net Net-(JP107-A): track 0.00 -> 12.5 mm
- net In3L: track 0.00 -> 10.7 mm
- net In2L: track 0.00 -> 10.5 mm
- net Net-(C106-Pad2): track 0.00 -> 5.40 mm
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- added copper zone on B.Cu, net GND
- added copper zone on F.Cu, net GND
Other:
- board text added: "Johansen Engineering PocketOperator_TDA1308AMP 26/11-2025 Rev A"
